File: Fugu2.kicad_pcb (KiCad board)
At the start: 2 copper layers, 50 x 80 mm, 108 parts, among them J1 Conn_02x03_ESP_PROG, J10 SOLAR, J2 I2C Conn, J3 Conn_L_SW, J4 MCU head, J6 Conn_L_out, J7 3.3V PSU, J8 12V PSU, J9 BAT, Q1 IPP055N08NF2SAKMA1, Q2 FDPF2D3N10C, Q3 IPP055N08NF2SAKMA1, Q4 BSS123, Q5 TPH1R306PL,L1Q, Q6 TPH1R306PL,L1Q, Q7 TPH1R306PL,L1Q, U1 UCC21330BQDRQ1, U2 ESP32-S3-WROOM-1, U3 INA226

Commit message: First cut, with refactored schematic (PCB now busted, it's a WIP)
Parts:
- removed C21, C22: 10uF, 100V, X7S, Capacitor_SMD:C_2220_5650Metric
- removed D16: ST15100S, open-pe:TO-277B_ThermalVias
- removed D3, D4, D5: LESD5D5.0CT1G, Diode_SMD:D_SOD-523
- removed D9: ST40100C, open-pe:TO-220-3_Horizontal_BottomHeatsink_NoHole
- removed DZ1: SM2T3V3A, PCM_Diode_SMD_AKL:D_Powermite_KA
- removed J2: I2C Conn, Connector_PinSocket_2.00mm:PinSocket_1x04_P2.00mm_Vertical
- removed J6: Conn_L_out, open-pe:SolderWire-1x01_D3.5mm
- removed J7: 3.3V PSU, Connector_PinHeader_2.54mm:PinHeader_1x03_P2.54mm_Vertical
- removed J8: 12V PSU, Connector_PinHeader_2.54mm:PinHeader_1x03_P2.54mm_Vertical
- removed Q1: IPP055N08NF2SAKMA1, open-pe:TO-220-3_Horizontal_BottomHeatsink_SmallHole
- removed Q2: FDPF2D3N10C, open-pe:TO-220-3_Horizontal_BottomHeatsink_NoHole
- removed USB1: USBConn_01x04_Pin, Connector_PinHeader_2.54mm:PinHeader_1x04_P2.54mm_Vertical
- added C28: 1uF, 100V, X7S, Capacitor_SMD:C_0805_2012Metric_Pad1.18x1.45mm_HandSolder, F.Cu at (168.2, 46.1)
- added C29: 1uF, 100V, X7S, Capacitor_SMD:C_0805_2012Metric_Pad1.18x1.45mm_HandSolder, F.Cu at (168.2, 49.1)
- added C31: 220nF, 100V, X7S, Capacitor_SMD:C_0603_1608Metric_Pad1.08x0.95mm_HandSolder, F.Cu at (156.4, 64.9)
- added C32: 2n2 50 V, Capacitor_SMD:C_0805_2012Metric_Pad1.18x1.45mm_HandSolder, F.Cu at (168.2, 52.1)
- added C33: 56pF 50V, Capacitor_SMD:C_0603_1608Metric_Pad1.08x0.95mm_HandSolder, F.Cu at (156.4, 67.4)
- added C34: 2n2 100 V, Capacitor_SMD:C_0805_2012Metric_Pad1.18x1.45mm_HandSolder, F.Cu at (168.2, 55.1)
- added C35: 22uF 25V X7R, Capacitor_SMD:CP_Elec_6.3x5.9, F.Cu at (180.3, 48.6)
- added C36: 1uF, 100V, X7S, Capacitor_SMD:C_0805_2012Metric_Pad1.18x1.45mm_HandSolder, F.Cu at (161.8, 160.6)
- added C37: 1uF, 100V, X7S, Capacitor_SMD:C_0805_2012Metric_Pad1.18x1.45mm_HandSolder, F.Cu at (161.8, 163.6)
- added C38: 220nF, 100V, X7S, Capacitor_SMD:C_0603_1608Metric_Pad1.08x0.95mm_HandSolder, F.Cu at (150.0, 172.4)
- added C39: 2n2 50 V, Capacitor_SMD:C_0805_2012Metric_Pad1.18x1.45mm_HandSolder, F.Cu at (161.8, 166.6)
- added C41: 56pF 50V, Capacitor_SMD:C_0603_1608Metric_Pad1.08x0.95mm_HandSolder, F.Cu at (150.0, 175.0)
- added C42: 2n2 100 V, Capacitor_SMD:C_0805_2012Metric_Pad1.18x1.45mm_HandSolder, F.Cu at (161.8, 169.7)
- added C43: 22uF 25V X7R, Capacitor_SMD:CP_Elec_6.3x5.9, F.Cu at (173.9, 159.3)
- added D17: MSS1P4-M3/89A, Diode_SMD:D_MicroSMP_AK, F.Cu at (151.0, 117.2)
- added J5: I2C, Connector_JST:JST_SH_SM04B-SRSS-TB_1x04-1MP_P1.00mm_Horizontal, F.Cu at (93.4, 26.7)
- added L1: L_Iron, Inductor_SMD:L_Sunlord_MWSA2213S, F.Cu at (7.75, 62.0)
- added L2: 100uH, Inductor_SMD:L_Taiyo-Yuden_NR-80xx_HandSoldering, F.Cu at (160.0, 49.4)
- added L3: 100uH, Inductor_SMD:L_Taiyo-Yuden_NR-80xx_HandSoldering, F.Cu at (153.6, 161.4)
- added R31: 0R, Resistor_SMD:R_0603_1608Metric, F.Cu at (44.9, 36.8)
- added R32: 0R, Resistor_SMD:R_0603_1608Metric, F.Cu at (44.9, 39.0)
- added R33: 0R, Resistor_SMD:R_0603_1608Metric, F.Cu at (45.0, 41.5)
- added R34: 7k5, Resistor_SMD:R_0805_2012Metric, F.Cu at (146.1, 129.1)
- added R38: 100k, Resistor_SMD:R_0805_2012Metric, F.Cu at (172.8, 46.0)
- added R39: ~, Resistor_SMD:R_0805_2012Metric, F.Cu at (172.8, 49.0)
- added R40: 33k, Resistor_SMD:R_0805_2012Metric, F.Cu at (172.8, 52.0)
- added R41: 10k, Resistor_SMD:R_0805_2012Metric, F.Cu at (172.8, 54.9)
- added R42: 100k, Resistor_SMD:R_0805_2012Metric, F.Cu at (166.4, 160.3)
- added R44: ~, Resistor_SMD:R_0805_2012Metric, F.Cu at (166.4, 163.3)
- added R45: 33k, Resistor_SMD:R_0805_2012Metric, F.Cu at (166.4, 166.2)
- added R46: 10k, Resistor_SMD:R_0805_2012Metric, F.Cu at (166.4, 169.2)
- added U5: USBLC6-2SC6, Package_TO_SOT_SMD:SOT-23-6, F.Cu at (94.1, 17.4)
- added U6: LM5163DDAR, Package_SO:HSOP-8-1EP_3.9x4.9mm_P1.27mm_EP2.41x3.1mm_ThermalVias, F.Cu at (179.2, 64.2)
- added U7: LM5163DDAR, Package_SO:HSOP-8-1EP_3.9x4.9mm_P1.27mm_EP2.41x3.1mm_ThermalVias, F.Cu at (172.8, 173.3)
- C10, C11, C12: value 470uF -> 470u
- C13: value 47uF, 100V -> 47u 100V
- C14: value 100nF, 100V -> 100n 100V
- C15: value 100nF, 25V -> 100n 25V; moved to F.Cu
- C16: value 1uF, 100V, X7S -> 1u 100V X7S; moved to F.Cu
- C17, C18: value 220nF, 100V, X7S -> 220n 100V X7S; moved to F.Cu
- C19: value 10uF, 16V -> 10u 16V
- C2, C24, C4: value 100nF, 25V -> 100n 25V
- C20, C23: value 10nF, 50V -> 10n 50V
- C25, C3: value 470nF, 25V -> 470n 25V
- C27, C9: value 1uF, 100V, X7S -> 1u 100V X7S
- C6, C7: value 100nF, X7R, 25V -> 100n 25V X7R
- C8: value 2.2nF, 200V, X7S -> 2.2n 200V X7S
- J3: value Conn_L_SW -> USB_C_Receptacle_USB2.0_14P; footprint open-pe:SolderWire-1x01_D3.5mm -> afork-kicad-parts:USB-C-SMD_G-SWITCH_GT-USB-7010ASV
- Q3: footprint open-pe:TO-220-3_Horizontal_BottomHeatsink_SmallHole -> Package_TO_SOT_THT:TO-220-3_Vertical; moved to F.Cu
- R10, R4, R6: value 4.7 -> 4R7
- R11: value 7.5 -> 7R5
- R13, R14: value 10k -> 4k7
- R16, R18, TH1: moved to F.Cu
- R19: value 20 -> 20R
- R20: value 7.5k -> 7k5; moved to F.Cu
- R25, R27: value 22 -> 22R
- R26: value 0.0005 -> 0R0005
- R28, R29: value 47k, 1% -> 47k 1%
- R5, R7: value 0 -> 0R
- R8, R9: value 7.5k -> 7k5
- U2: footprint open-pe:ESP32-S3-WROOM-1-noPIN15 -> RF_Module:ESP32-S3-WROOM-1
- moved C5 144.9 mm to (170.3, 108.6), turned to 0 degrees
- moved R12 137.3 mm to (164.6, 111.9)
- moved D1 136.7 mm to (151.0, 114.3), turned to 0 degrees
- moved R9 132.4 mm to (146.1, 123.2), turned to 0 degrees
- moved R7 131.7 mm to (146.1, 117.3), turned to 0 degrees
- moved C8 130.4 mm to (169.8, 111.8), turned to 0 degrees
- moved Q3 130.0 mm to (151.5, 110.9)
- moved R6 129.9 mm to (146.1, 114.3), turned to 0 degrees
- moved R10 129.9 mm to (146.1, 126.1)
- moved R5 129.8 mm to (146.1, 111.4), turned to 0 degrees
- moved R11 128.0 mm to (164.6, 108.6)
- moved R4 125.3 mm to (146.1, 108.4), turned to 0 degrees
- moved R8 120.0 mm to (146.1, 120.2), turned to 0 degrees
- moved TPA1 114.1 mm to (163.3, 120.0)
- moved C27 113.9 mm to (139.6, 102.6), turned to 0 degrees
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Connections:
- net +3.3V renamed +3V3
- net ADC_Vin renamed /uC/ADC_Vin
- net ALERT renamed /uC/ALERT
- net BflowG renamed Net-(DZ2-K)
- net BflowSD renamed /uC/BFlowSD
- net HO renamed /GateDrive/HI
- net IO0 renamed /uC/IO0
- net LED renamed /uC/LED
- net LO renamed /GateDrive/LO
- net NTC renamed /uC/NTC
- net RX renamed /uC/RX
- net SCL renamed /uC/SCL
- net SDA renamed /uC/SDA
- net TX renamed /uC/TX
- C10 pad 1: BflowS -> /backflow/BFLOWS
- C20 pad 2: BflowS -> Bat+
- C3 pad 1: GND -> /uC/EN
- C3 pad 2: EN -> GND
- C8 pad 2: BuckGND -> /snubber/BUCKGND
- D7 pad 2: Vusb -> /PowerSupply/Vusb
- DZ2 pad 1: BflowS -> Bat+
- J1 pad 1: EN -> /uC/EN
- J4 pad 10: INH -> /uC/INL
- J4 pad 12: SD -> /uC/INH
- J4 pad 14: INL -> /uC/SD
- Q5 pad 1: BflowS -> Bat+
- Q5 pad 3: Bat+ -> /backflow/BFLOWS
- Q6 pad 1: BflowS -> Bat+
- Q6 pad 3: Bat+ -> /backflow/BFLOWS
- Q7 pad 1: BflowS -> Bat+
- Q7 pad 3: Bat+ -> /backflow/BFLOWS
- R11 pad 1: SW -> /snubber/SW
- R12 pad 2: SW -> /snubber/SW
- R2 pad 2: EN -> /uC/EN
- R24 pad 1: BflowS -> Bat+
- R5 pad 2: Net-(D1-A) -> Net-(D17-A)
- TPINH1 pad 1: INH -> /uC/INH
- TPINL1 pad 1: INL -> /uC/INL
- TPSD1 pad 1: SD -> /uC/SD
- U1 pad 1: INL -> Net-(U1-INA)
- U1 pad 2: INH -> Net-(U1-INB)
- U1 pad 5: SD -> Net-(U1-DIS)
- U2 pad 13: USB_D- -> /uC/USB_N
- U2 pad 14: USB_D+ -> /uC/USB_P
- U2 pad 22: INL -> /uC/INL
- U2 pad 23: INH -> /uC/INH
- U2 pad 24: SD -> /uC/SD
- U2 pad 3: EN -> /uC/EN
- U2 pad 5: Net-(U2-GPIO5/TOUCH5/ADC1_CH4) -> unconnected-(U2-GPIO5/TOUCH5/ADC1_CH4-Pad5)
- U2 pad 6: Net-(U2-GPIO6/TOUCH6/ADC1_CH5) -> unconnected-(U2-GPIO6/TOUCH6/ADC1_CH5-Pad6)
- bfs1 pad 1: BflowS -> Bat+
Routing:
- net /uC/LED: track 63.9 -> 0.00 mm
- net +3V3: track 202.4 -> 144.9 mm, vias 4 -> 3
- net Solar+: track 99.4 -> 42.7 mm
- net /uC/ADC_Vin: track 17.3 -> 64.4 mm, vias 1 -> 2
- net /uC/RX: track 39.2 -> 1.40 mm, vias 0 -> 2
- net /uC/TX: track 39.5 -> 2.05 mm, vias 0 -> 2
- net (no net): track 0.00 -> 35.1 mm, vias 0 -> 1
- net SD: track 33.7 -> 0.00 mm
- net EN: track 33.2 -> 0.00 mm
- net INH: track 32.1 -> 0.00 mm
- net /uC/IO0: track 37.1 -> 6.15 mm
- net Vusb: track 28.3 -> 0.00 mm
- net INL: track 23.0 -> 0.00 mm
- net /uC/SCL: track 71.3 -> 48.7 mm
- net /uC/NTC: track 27.9 -> 9.60 mm
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- added copper zone on B.Cu, net /backflow/BFLOWS
- added copper zone on F.Cu, net /backflow/BFLOWS
- removed copper zone on B.Cu, net BflowS
- removed copper zone on F.Cu, net BflowS
Other:
- board size 50 x 80 mm -> 100 x 100 mm
