File: icaps.kicad_sch (KiCad schematic)
At the start: 9 parts

Commit message: Mega-cleanup
Parts:
- C16, C27, C9: LCSC HMK212BC7105KGHTE -> (none)
- C17, C18: LCSC HMK107C7224KAHTE -> (none)
- C21, C22: footprint Capacitor_SMD:C_2220_5650Metric -> Capacitor_SMD:C_1210_3225Metric; LCSC GRM32EC72A106KE05L -> C576517; Manufacturer (none) -> Murata
Changed lines of the file:
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@@
 			)
 		)
-		(property "LCSC" "HMK107C7224KAHTE"
+		(property "LCSC" ""
 			(at 171.45 92.71 0)
 			(effects
@@
 			)
 		)
-		(property "LCSC" "HMK212BC7105KGHTE"
+		(property "LCSC" ""
 			(at 152.4 85.09 0)
 			(effects
@@
 			)
 		)
-		(property "Footprint" "Capacitor_SMD:C_2220_5650Metric"
+		(property "Footprint" "Capacitor_SMD:C_1210_3225Metric"
 			(at 135.5852 96.52 0)
 			(effects
@@
 			)
 		)
-		(property "Manufacturer" ""
+		(property "Manufacturer" "Murata"
 			(at 134.62 92.71 0)
 			(effects
@@
 			)
 		)
-		(property "LCSC" "GRM32EC72A106KE05L"
+		(property "LCSC" "C576517"
 			(at 134.62 92.71 0)
 			(effects
@@
 			)
 		)
-		(property "LCSC" "HMK212BC7105KGHTE"
+		(property "LCSC" ""
 			(at 146.05 85.09 0)
 			(effects
@@
 			)
 		)
-		(property "Footprint" "Capacitor_SMD:C_2220_5650Metric"
+		(property "Footprint" "Capacitor_SMD:C_1210_3225Metric"
 			(at 140.6652 96.52 0)
 			(effects
@@
 			)
 		)
-		(property "Manufacturer" ""
+		(property "Manufacturer" "Murata"
 			(at 139.7 92.71 0)
 			(effects
@@
 			)
 		)
-		(property "LCSC" "GRM32EC72A106KE05L"
+		(property "LCSC" "C576517"
 			(at 139.7 92.71 0)
 			(effects
@@
 			)
 		)
-		(property "LCSC" "HMK107C7224KAHTE"
+		(property "LCSC" ""
 			(at 165.1 92.71 0)
 			(effects
@@
 			)
 		)
-		(property "LCSC" "HMK212BC7105KGHTE"
+		(property "LCSC" ""
 			(at 158.75 85.09 0)
 			(effects
