File: inverter.kicad_sch (KiCad schematic)
At the start: 16 parts, among them Q1 IPP055N08NF2SAKMA1, Q2 FDPF2D3N10C, Q3 IPP055N08NF2SAKMA1

Commit message: Mega-cleanup
Parts:
- D16: value ST15100S -> SP15100L; footprint open-pe:TO-277B_ThermalVias -> local:TO-277B-AAK; symbol open-pe:ST15100S -> Device:D_Schottky_AAK; LCSC (none) -> C5375261; MPN ST15100S -> (none); Manufacturer SMC -> XCH
- D9: value ST40100C -> MBR20100CT; footprint open-pe:TO-220-3_Horizontal_BottomHeatsink_NoHole -> Package_TO_SOT_THT:TO-220-3_Vertical; LCSC (none) -> C173465
- Q1: footprint open-pe:TO-220-3_Horizontal_BottomHeatsink_SmallHole -> local:TO-220-3_Horizontal_TabUp-nohole; Desc HS -> (none)
- Q2: value FDPF2D3N10C -> IPP055N08NF2SAKMA1; footprint open-pe:TO-220-3_Horizontal_BottomHeatsink_NoHole -> local:TO-220-3_Horizontal_TabUp-nohole; Desc LS -> (none)
- Q3: footprint Package_TO_SOT_THT:TO-220-3_Vertical -> local:TO-220-3_Horizontal_TabUp-nohole; Desc HS -> (none)
Connections:
- net BuckGND: now also D16.1 (A), D16.2 (A); no longer D16.A
- net SW: now also D16.3 (K); no longer D16.K
Other:
- note added: "was: SMC ST15100S"
- note added: "was: ST40100C"
