File: snubber.kicad_sch (KiCad schematic)
At the start: 4 parts

Commit message: Mega-cleanup
Connections:
- net BUCKGND renamed BuckGND
Changed lines of the file:
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@@
+		)
+	)
+	(global_label "BuckGND"
+		(shape input)
+		(at 125.73 100.33 0)
+		(fields_autoplaced yes)
+		(effects
+			(font
+				(size 1.27 1.27)
+			)
+			(justify left)
+		)
+		(property "Intersheetrefs" "${INTERSHEET_REFS}"
+			(at 137.1214 100.33 0)
+			(effects
+				(font
+					(size 1.27 1.27)
+				)
+				(justify left)
+				(hide yes)
+			)
 		)
 	)
 	(global_label "Solar+"
-		(shape passive)
+		(shape input)
 		(at 123.19 66.04 0)
 		(fields_autoplaced yes)
@@
 		)
 		(property "Intersheetrefs" "${INTERSHEET_REFS}"
-			(at 131.5952 66.04 0)
+			(at 132.7065 66.04 0)
 			(effects
 				(font
@@
 		)
 	)
-	(hierarchical_label "BUCKGND"
-		(shape input)
-		(at 125.73 100.33 0)
-		(effects
-			(font
-				(size 1.27 1.27)
-			)
-			(justify left)
-		)
-	)
