File: PowerSupply.kicad_sch (KiCad schematic)
At the start: 10 parts, among them J7 3.3V PSU, J8 12V PSU, P1 USB4105-GF-A

Commit message: First cut, with refactored schematic (PCB now busted, it's a WIP)
Parts:
- removed J7: 3.3V PSU, Connector_PinHeader_2.54mm:PinHeader_1x03_P2.54mm_Vertical, symbol Connector:Conn_01x03_Socket
- removed J8: 12V PSU, Connector_PinHeader_2.54mm:PinHeader_1x03_P2.54mm_Vertical, symbol Connector:Conn_01x03_Socket
- removed P1: USB4105-GF-A, symbol Connector:USB_C_Plug_USB2.0
- added C28, C29, C36, C37: 1uF, 100V, X7S, Capacitor_SMD:C_0805_2012Metric_Pad1.18x1.45mm_HandSolder, symbol Device:C_Small
- added C30, C40: 470p, Capacitor_SMD:C_0603_1608Metric, symbol Device:C_Small
- added C31, C38: 220nF, 100V, X7S, Capacitor_SMD:C_0603_1608Metric_Pad1.08x0.95mm_HandSolder, symbol Device:C_Small
- added C32, C39: 2n2 50 V, Capacitor_SMD:C_0805_2012Metric_Pad1.18x1.45mm_HandSolder, symbol Device:C_Small
- added C33, C41: 56pF 50V, Capacitor_SMD:C_0603_1608Metric_Pad1.08x0.95mm_HandSolder, symbol Device:C_Small
- added C34, C42: 2n2 100 V, Capacitor_SMD:C_0805_2012Metric_Pad1.18x1.45mm_HandSolder, symbol Device:C_Small
- added C35, C43: 22uF 25V X7R, Capacitor_SMD:CP_Elec_6.3x5.9, symbol Device:C_Polarized
- added L2, L3: 100uH, Inductor_SMD:L_Taiyo-Yuden_NR-80xx_HandSoldering, symbol Device:L
- added R37, R43: 22, Resistor_SMD:R_0603_1608Metric, symbol Device:R_Small
- added R38, R42: 100k, Resistor_SMD:R_0805_2012Metric, symbol Device:R_Small
- added R39, R44: ~, Resistor_SMD:R_0805_2012Metric, symbol Device:R_Small
- added R40, R45: 33k, Resistor_SMD:R_0805_2012Metric, symbol Device:R_Small
- added R41, R46: 10k, Resistor_SMD:R_0805_2012Metric, symbol Device:R_Small
- added U6, U7: LM5163DDAR, Package_SO:HSOP-8-1EP_3.9x4.9mm_P1.27mm_EP2.41x3.1mm_ThermalVias, symbol Regulator_Switching:LM5164DDA
- C13: value 47uF, 100V -> 47u 100V
- DZ1: now not fitted; now left out of the parts list
Connections:
- net +12V: now also C34.2, C35.1, L2.2, R40.1
- net +3.3V: now also C42.2, C43.1, L3.2, R45.1; no longer DZ1.1 (K)
- net GND: now also C28.2, C29.2, C30.2, C31.2, C35.2, C36.2, C37.2, C38.2, C40.2, C43.2, R38.2, R41.2, R42.2, R46.2, U6.1 (GND), U6.9 (EP), U7.1 (GND), U7.9 (EP)
- net at C13.1, D13.1 (K), D7.1 (K)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: now also C28.1, C29.1, C31.1, C36.1, C37.1, C38.1, U6.2 (VIN), U6.3 (EN/UVLO), U7.2 (VIN), U7.3 (EN/UVLO)
- new net: C33.1, R40.2, R41.1, U6.5 (FB)
- new net: C33.2, C34.1, R39.2
- new net: C39.2, L3.1, R43.1, R44.1, U7.8 (SW)
- new net: C41.2, C42.1, R44.2
- new net: C41.1, R45.2, R46.1, U7.5 (FB)
- new net: C30.1, R37.2
- new net: C32.1, U6.7 (BST)
- new net: C32.2, L2.1, R37.1, R39.1, U6.8 (SW)
- new net: R38.1, U6.4 (RON)
- new net: R42.1, U7.4 (RON)
- new net: C39.1, U7.7 (BST)
- new net: C40.1, R43.2
- new net +3V3: DZ1.1 (K)
- no-connect marks 0 -> 2
Other:
- note added: "Bucks from: https://github.com/open-pe/buck100-LM5163"
- note added: "LM5163 100Vmax 0.5A LM5164 100Vmax 1.0A LM5168 120Vmax 0.3A LM5169 120Vmax 0.65A"
- note added: "Snubber"
- note added: "TI Design Tool"
- note removed: "esp32 has wifi. we will need usb mostly for dev, jtag, hw config. system integration through usb is rather uncommon and usb hosts usually have bluetooth. we can also put the esp32 i host mode and use a female connector for usb sticks etc. to keep things simple & small, we chose for a 2.54 4-pin header connector (TOOD JST?) the USB connector enables - flashing/programming and serial console - JTAG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"
- note removed: "open-pe/buck80-XL7005A"
- note removed: "see esp-rust-board for footprint"
- moved on the sheet: C13, D11, D12, D13, D7, F2

Commit message: Mega-cleanup
Parts:
- C13: LCSC ERS1KM470F12OT -> (none); MPN 47uF, 100V -> ERS1KM470F12OT
- C30, R37: now in the parts list
- C32, C34, C39, C42: MPN (none) -> GCM155R71H222KA37D; Ref GCM155R71H222KA37D -> (none)
- D7: now not fitted
- L2, L3: footprint Inductor_SMD:L_Taiyo-Yuden_NR-80xx_HandSoldering -> local:IND-SMD_L8.0-W8.0; LCSC (none) -> C223045; Manufacturer (none) -> Taiyo Yuden
Other:
- moved on the sheet: C34, C42, L2, L3, R39, R44

Commit message: Increased resistor sizes from 0603 to 0805
Parts:
- C40: now in the parts list
- R37: footprint Resistor_SMD:R_0603_1608Metric -> Resistor_SMD:R_0805_2012Metric
- R43: footprint Resistor_SMD:R_0603_1608Metric -> Resistor_SMD:R_0805_2012Metric; now in the parts list
Changed lines of the file:
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@@
 		(unit 1)
 		(exclude_from_sim no)
-		(in_bom no)
-		(on_board no)
+		(in_bom yes)
+		(on_board yes)
 		(dnp yes)
 		(fields_autoplaced yes)
@@
 		(unit 1)
 		(exclude_from_sim no)
-		(in_bom no)
-		(on_board no)
+		(in_bom yes)
+		(on_board yes)
 		(dnp yes)
 		(fields_autoplaced yes)
@@
 			)
 		)
-		(property "Footprint" "Resistor_SMD:R_0603_1608Metric"
+		(property "Footprint" "Resistor_SMD:R_0805_2012Metric"
 			(at 182.88 127 0)
 			(effects
@@
 			)
 		)
-		(property "Footprint" "Resistor_SMD:R_0603_1608Metric"
+		(property "Footprint" "Resistor_SMD:R_0805_2012Metric"
 			(at 182.88 69.85 0)
 			(effects
