File: Fugu2.kicad_sch (KiCad schematic)
At the start: 62 parts, among them J10 SOLAR, J3 Conn_L_SW, J6 Conn_L_out, J9 BAT, Q1 IPP055N08NF2SAKMA1, Q2 FDPF2D3N10C, Q3 IPP055N08NF2SAKMA1, Q5 TPH1R306PL,L1Q, Q6 TPH1R306PL,L1Q, Q7 TPH1R306PL,L1Q, U3 INA226

Commit message: First cut, with refactored schematic (PCB now busted, it's a WIP)
Parts:
- removed C11: 470uF, Capacitor_THT:CP_Radial_D16.0mm_P7.50mm, symbol Device:C_Polarized
- removed C12: 470uF, Capacitor_THT:CP_Radial_D18.0mm_P7.50mm, symbol Device:C_Polarized
- removed C15, C24: 100nF, 25V, Capacitor_SMD:C_0805_2012Metric, symbol Device:C_Small
- removed C16, C27, C9: 1uF, 100V, X7S, Capacitor_SMD:C_0805_2012Metric, symbol Device:C
- removed C17, C18: 220nF, 100V, X7S, Capacitor_SMD:C_0603_1608Metric, symbol Device:C
- removed C21, C22: 10uF, 100V, X7S, Capacitor_SMD:C_2220_5650Metric, symbol Device:C
- removed C23: 10nF, 50V, Capacitor_SMD:C_0805_2012Metric, symbol Device:C_Small
- removed C25: 470nF, 25V, Capacitor_SMD:C_0805_2012Metric, symbol Device:C_Small
- removed C5: 2.2nF, 200V, X7S, Capacitor_SMD:C_1206_3216Metric, symbol Device:C_Small
- removed C8: 2.2nF, 200V, X7S, Capacitor_SMD:C_0805_2012Metric_Pad1.18x1.45mm_HandSolder, symbol Device:C_Small
- removed D1: MSS1P4-M3/89A, Diode_SMD:D_MicroSMP_AK, symbol Device:D_Small
- removed D14: MSS1P4, Diode_SMD:D_SMF, symbol Device:D_Small
- removed D16: ST15100S, open-pe:TO-277B_ThermalVias, symbol open-pe:ST15100S
- removed D2: WS2812B, LED_SMD:LED_WS2812B_PLCC4_5.0x5.0mm_P3.2mm, symbol LED:WS2812B
- removed D6: LESD5D5.0CT1G, Diode_SMD:D_SOD-523, symbol PCM_Diode_TVS_AKL:D_TVS_Bidirectional_Generic
- removed D9: ST40100C, open-pe:TO-220-3_Horizontal_BottomHeatsink_NoHole, symbol Device:D_Dual_CommonCathode_AKA_Parallel
- removed J3: Conn_L_SW, open-pe:SolderWire-1x01_D3.5mm, symbol Connector:Conn_01x01_Socket
- removed J6: Conn_L_out, open-pe:SolderWire-1x01_D3.5mm, symbol Connector:Conn_01x01_Socket
- removed L1: L, open-pe:Fuse_Blade_Mini_directSolder_noSlots, symbol Device:L
- removed Q1, Q3: IPP055N08NF2SAKMA1, open-pe:TO-220-3_Horizontal_BottomHeatsink_SmallHole, symbol Transistor_FET:IPP060N06N
- removed Q2: FDPF2D3N10C, open-pe:TO-220-3_Horizontal_BottomHeatsink_NoHole, symbol Transistor_FET:IPP060N06N
- removed Q5, Q6, Q7: TPH1R306PL,L1Q, open-pe:Infineon_PG-TDSON-8_FL, symbol open-pe:HYG025N06LS1C2
- removed R10, R4, R6: 4.7, Resistor_SMD:R_0805_2012Metric, symbol Device:R_Small
- removed R11, R12: 7.5, Resistor_SMD:R_1206_3216Metric, symbol Device:R_Small
- removed R16: 10k, Resistor_SMD:R_0805_2012Metric, symbol Device:R_Small
- removed R18: 200k, Resistor_SMD:R_0805_2012Metric, symbol Device:R_Small
- removed R20, R8, R9: 7.5k, Resistor_SMD:R_0805_2012Metric, symbol Device:R_Small
- removed R25, R27: 22, Resistor_SMD:R_0805_2012Metric, symbol Device:R_Small
- removed R28, R29: 47k, 1%, Resistor_SMD:R_0805_2012Metric, symbol Device:R_Small
- removed R5, R7: 0, Resistor_SMD:R_0805_2012Metric, symbol Device:R_Small
- removed TH1: NCP18XH103F03RB, Resistor_SMD:R_0603_1608Metric_Pad0.98x0.95mm_HandSolder, symbol Device:Thermistor_NTC
- removed U3: INA226, Package_SO:VSSOP-10_3x3mm_P0.5mm, symbol Sensor_Energy:INA226
- added L1: L_Iron, Inductor_SMD:L_Sunlord_MWSA2213S, symbol Device:L_Iron
- C10: value 470uF -> 470u
- C14: value 100nF, 100V -> 100n 100V
- R26: value 0.0005 -> 0R0005
Connections:
- net SW: now also L1.1
- net BflowS renamed backflow/BFLOWS
- net backflow/BFLOWS: now also L1.2
- no-connect marks 1 -> 0
Other:
- added sheet backflow (backflow.kicad_sch)
- added sheet csense (csense.kicad_sch)
- added sheet icaps (icaps.kicad_sch)
- added sheet inverter (inverter.kicad_sch)
- added sheet snubber (snubber.kicad_sch)
- sheet GateDrive ports: added HI, INH, INL, LO, SD, SW; removed none
- sheet PowerSupply ports: added Vusb; removed none
- sheet uC ports: added ALERT, BFlowSD, INH, INL, SCL, SD, SDA, Vusb; removed none
- note added: "Why current senser here? Because: - Low side is simpler - ~0V common mode -> can use ina226 @ 48V battery - MCU ground should be bat(-) for wired interfaces"
- note removed: "ADC max: 2.45V"
- note removed: "INA226: 36V 16bit bi-dir place-in alternatives: INA230 (36V 16bit, higher error) INA220 (26V 12bit, no ALERT => NC) INA228 (85V 20bit)"
- note removed: "We need the Solar Voltage for OV/UV detection and synchronous recitification (diode emulation)"
- note removed: "Why current senser here? - Low side is simpler - ~0V common mode -> can use ina226 @ 48V battery - MCU ground should be bat(-) for wired interfaces"
- note removed: "alternativse in 8-power* housing (Rdson(max)@25°C,10V): TPH1R306PL,L1Q (60V 1.3mΩ) SiR626LDP (60V, 1.5m) AONS66612 (60V 1.65mΩ) HYG025N06LS1C2 (60V, 2.1mΩ) TPHR6503PL,L1Q (30V 0.6mΩ) TPHR9003NL1,LQ (30V 0.9mΩ) AON6500 (30V 0.95mΩ) AONS32302 (30v 1.35mΩ) AONS32311"
- note removed: "f_c=1/(2pi*R20*C15) f_c=221Hz"
- note removed: "fc_U=677Hz too low? fc_I="
- note removed: "snubber circuits"
- moved on the sheet: C1, C10, C14, F1, H1, H2, H3, H4, H5, H6, J10, J9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

Commit message: Mega-cleanup
Parts:
- F1: footprint open-pe:Fuse_Blade_ATO_directSolderThin -> afork-kicad-parts:FUSE-TH_XF-506P
- J10, J9: footprint TerminalBlock_MetzConnect:TerminalBlock_MetzConnect_Type703_RT10N02HGLU_1x02_P9.52mm_Horizontal -> local:CONN-TH_DG135T-10.16-02P-14-00A; LCSC (none) -> C2981775; MPN DNP -> DB135-10.16-2P-GN-P; Manufacturer (none) -> DORABO
- L1: value L_Iron -> RSEQ32-470M; footprint Inductor_SMD:L_Sunlord_MWSA2213S -> local:IND-TH_L33.0-W31.5; LCSC (none) -> C37634010; Manufacturer (none) -> Ruishen
Other:
- moved on the sheet: H2, H3, H4, H5, H6

Commit message: Removed parts from open-pe
Parts:
- J10, J9: symbol open-pe:Screw_TerminalBlock_WR-TBL_2566_01x02 -> Connector:Screw_Terminal_01x02
- R26: footprint open-pe:R_2512_6332Metric_Pad2.72x3.40mm_HandSolder -> Resistor_SMD:R_2512_6332Metric_Pad1.40x3.35mm_HandSolder; Manufacturer (none) -> Milliohm
Changed lines of the file:
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@@
 	)
 	(symbol
-		(lib_id "open-pe:Screw_TerminalBlock_WR-TBL_2566_01x02")
+		(lib_id "Connector:Screw_Terminal_01x02")
 		(at 48.26 76.2 0)
 		(mirror y)
@@
 			)
 		)
-		(property "Description" ""
+		(property "Description" "Generic screw terminal, single row, 01x02, script generated (kicad-library-utils/schlib/autogen/connector/)"
 			(at 48.26 76.2 0)
 			(effects
@@
 			)
 		)
-		(property "Footprint" "open-pe:R_2512_6332Metric_Pad2.72x3.40mm_HandSolder"
+		(property "Footprint" "Resistor_SMD:R_2512_6332Metric_Pad1.40x3.35mm_HandSolder"
 			(at 203.2 99.06 0)
 			(effects
@@
 			)
 		)
-		(property "Manufacturer" ""
+		(property "Manufacturer" "Milliohm"
 			(at 203.2 99.06 0)
 			(effects
@@
 	)
 	(symbol
-		(lib_id "open-pe:Screw_TerminalBlock_WR-TBL_2566_01x02")
+		(lib_id "Connector:Screw_Terminal_01x02")
 		(at 237.49 85.09 0)
 		(mirror x)
@@
 			)
 		)
-		(property "Description" ""
+		(property "Description" "Generic screw terminal, single row, 01x02, script generated (kicad-library-utils/schlib/autogen/connector/)"
 			(at 237.49 85.09 0)
 			(effects

Commit message: Added value for fuse (comes from upstream)
Parts:
- F1: value Fuse -> 40A
Changed lines of the file:
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@@
 			)
 		)
-		(property "Value" "Fuse"
+		(property "Value" "40A"
 			(at 226.06 68.6378 90)
 			(effects
