File: backflow.kicad_sch (KiCad schematic)
At the start: 13 parts, among them Q4 BSS123, Q5 TPH1R306PL,L1Q, Q6 TPH1R306PL,L1Q, Q7 TPH1R306PL,L1Q

Commit message: Mega-cleanup
Parts:
- Q5, Q6, Q7: value TPH1R306PL,L1Q -> NTMFS5C612NLT1G; footprint open-pe:Infineon_PG-TDSON-8_FL -> local:DFN-5_L6.1-W5.1-P1.27-BL; LCSC (none) -> C348543; MPN TPH1R306PL,L1Q -> NTMFS5C612NLT1G

Commit message: Removed parts from open-pe
Parts:
- Q5, Q6, Q7: symbol open-pe:HYG025N06LS1C2 -> Transistor_FET:Q_NMOS_SSSGD_AvalancheRated
Connections:
- net BFLOWD: now also Q5.2 (S), Q6.2 (S), Q7.2 (S)
- net BFLOWS: now also Q5.5 (D), Q6.5 (D), Q7.5 (D); no longer Q5.3 (S), Q6.3 (S), Q7.3 (S)
- net at C20.1, DZ2.3 (K), R21.1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: now also Q5.4 (G), Q6.4 (G), Q7.4 (G); no longer Q5.2 (S), Q6.2 (S), Q7.2 (S)
Changed lines of the file:
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@@
 	)
 	(symbol
-		(lib_name "HYG025N06LS1C2_2")
-		(lib_id "open-pe:HYG025N06LS1C2")
+		(lib_id "Transistor_FET:Q_NMOS_SSSGD_AvalancheRated")
 		(at 118.11 85.09 0)
 		(unit 1)
@@
 		)
 		(property "Footprint" "local:DFN-5_L6.1-W5.1-P1.27-BL"
-			(at 123.19 86.995 0)
-			(effects
-				(font
-					(size 1.27 1.27)
-				)
-				(justify left)
-				(hide yes)
-			)
-		)
-		(property "Datasheet" "https://www.lcsc.com/datasheet/C348543.pdf"
-			(at 118.11 85.09 90)
-			(effects
-				(font
-					(size 1.27 1.27)
-				)
-				(justify left)
-				(hide yes)
-			)
-		)
-		(property "Description" ""
+			(at 123.19 82.55 0)
+			(effects
+				(font
+					(size 1.27 1.27)
+				)
+				(hide yes)
+			)
+		)
+		(property "Datasheet" "~"
+			(at 118.11 85.09 0)
+			(effects
+				(font
+					(size 1.27 1.27)
+				)
+				(hide yes)
+			)
+		)
+		(property "Description" "N-MOSFET transistor, source (pins 1-3)/gate/drain (pin 5), SO-8/SO-8F/SO-8FL/SON-8/PowerPAK-8/TDSON-8/VSON-8"
 			(at 118.11 85.09 0)
 			(effects
@@
 		(pin "1"
 		)
+		(pin "4"
+		)
 		(pin "2"
 		)
-		(pin "2"
-		)
 		(pin "3"
 		)
-		(pin "3"
+		(pin "5"
 		)
 		(instances
@@
 	)
 	(symbol
-		(lib_name "HYG025N06LS1C2_1")
-		(lib_id "open-pe:HYG025N06LS1C2")
+		(lib_id "Transistor_FET:Q_NMOS_SSSGD_AvalancheRated")
 		(at 152.4 85.09 0)
 		(unit 1)
@@
 		)
 		(property "Footprint" "local:DFN-5_L6.1-W5.1-P1.27-BL"
-			(at 157.48 86.995 0)
-			(effects
-				(font
-					(size 1.27 1.27)
-				)
-				(justify left)
-				(hide yes)
-			)
-		)
-		(property "Datasheet" "https://www.lcsc.com/datasheet/C348543.pdf"
-			(at 152.4 85.09 90)
-			(effects
-				(font
-					(size 1.27 1.27)
-				)
-				(justify left)
-				(hide yes)
-			)
-		)
-		(property "Description" ""
+			(at 157.48 82.55 0)
+			(effects
+				(font
+					(size 1.27 1.27)
+				)
+				(hide yes)
+			)
+		)
+		(property "Datasheet" "~"
+			(at 152.4 85.09 0)
+			(effects
+				(font
+					(size 1.27 1.27)
+				)
+				(hide yes)
+			)
+		)
+		(property "Description" "N-MOSFET transistor, source (pins 1-3)/gate/drain (pin 5), SO-8/SO-8F/SO-8FL/SON-8/PowerPAK-8/TDSON-8/VSON-8"
 			(at 152.4 85.09 0)
 			(effects
@@
 		(pin "1"
 		)
+		(pin "5"
+		)
 		(pin "2"
 		)
-		(pin "2"
-		)
 		(pin "3"
 		)
-		(pin "3"
+		(pin "4"
 		)
 		(instances
@@
 	)
 	(symbol
-		(lib_id "open-pe:HYG025N06LS1C2")
+		(lib_id "Transistor_FET:Q_NMOS_SSSGD_AvalancheRated")
 		(at 137.16 85.09 0)
 		(unit 1)
@@
 		)
 		(property "Footprint" "local:DFN-5_L6.1-W5.1-P1.27-BL"
-			(at 142.24 86.995 0)
-			(effects
-				(font
-					(size 1.27 1.27)
-				)
-				(justify left)
-				(hide yes)
-			)
-		)
-		(property "Datasheet" "https://www.lcsc.com/datasheet/C348543.pdf"
-			(at 137.16 85.09 90)
-			(effects
-				(font
-					(size 1.27 1.27)
-				)
-				(justify left)
-				(hide yes)
-			)
-		)
-		(property "Description" ""
+			(at 142.24 82.55 0)
+			(effects
+				(font
+					(size 1.27 1.27)
+				)
+				(hide yes)
+			)
+		)
+		(property "Datasheet" "~"
+			(at 137.16 85.09 0)
+			(effects
+				(font
+					(size 1.27 1.27)
+				)
+				(hide yes)
+			)
+		)
+		(property "Description" "N-MOSFET transistor, source (pins 1-3)/gate/drain (pin 5), SO-8/SO-8F/SO-8FL/SON-8/PowerPAK-8/TDSON-8/VSON-8"
 			(at 137.16 85.09 0)
 			(effects
@@
 		(pin "1"
 		)
+		(pin "4"
+		)
 		(pin "2"
 		)
-		(pin "2"
-		)
 		(pin "3"
 		)
-		(pin "3"
+		(pin "5"
 		)
 		(instances

Commit message: Fixed orientation of backflow MOSFETs (thanks Fl4p!)
Connections:
- net BFLOWD: now also Q5.5 (D), Q6.5 (D), Q7.5 (D); no longer Q5.1 (S), Q5.2 (S), Q5.3 (S), Q6.1 (S), Q6.2 (S), Q6.3 (S), Q7.1 (S), Q7.2 (S), Q7.3 (S)
- net BFLOWS: now also Q5.1 (S), Q5.2 (S), Q5.3 (S), Q6.1 (S), Q6.2 (S), Q6.3 (S), Q7.1 (S), Q7.2 (S), Q7.3 (S); no longer Q5.5 (D), Q6.5 (D), Q7.5 (D)
Other:
- moved on the sheet: Q6, Q7
Changed lines of the file:
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@@
-	)
-	(junction
-		(at 128.27 91.44)
-		(diameter 0)
-		(color 0 0 0 0)
 	)
 	(junction
@@
 	)
 	(junction
+		(at 127 91.44)
+		(diameter 0)
+		(color 0 0 0 0)
+	)
+	(junction
 		(at 93.98 85.09)
 		(diameter 0)
@@
 	)
 	(junction
-		(at 154.94 97.79)
+		(at 151.13 97.79)
 		(diameter 0)
 		(color 0 0 0 0)
@@
 	)
 	(junction
-		(at 139.7 97.79)
+		(at 135.89 97.79)
 		(diameter 0)
 		(color 0 0 0 0)
 	)
 	(junction
-		(at 139.7 76.2)
+		(at 135.89 76.2)
 		(diameter 0)
 		(color 0 0 0 0)
@@
 	(wire
 		(pts
-			(xy 139.7 97.79) (xy 139.7 90.17)
+			(xy 135.89 97.79) (xy 135.89 90.17)
 		)
 		(stroke
@@
 	(wire
 		(pts
-			(xy 154.94 76.2) (xy 139.7 76.2)
+			(xy 151.13 76.2) (xy 135.89 76.2)
 		)
 		(stroke
@@
 	(wire
 		(pts
-			(xy 139.7 76.2) (xy 139.7 80.01)
-		)
-		(stroke
-			(width 0)
-			(type default)
-		)
-	)
-	(wire
-		(pts
-			(xy 120.65 76.2) (xy 139.7 76.2)
+			(xy 135.89 76.2) (xy 135.89 80.01)
+		)
+		(stroke
+			(width 0)
+			(type default)
+		)
+	)
+	(wire
+		(pts
+			(xy 120.65 76.2) (xy 135.89 76.2)
 		)
 		(stroke
@@
 	(wire
 		(pts
-			(xy 154.94 80.01) (xy 154.94 76.2)
+			(xy 151.13 80.01) (xy 151.13 76.2)
 		)
 		(stroke
@@
 	(wire
 		(pts
-			(xy 146.05 91.44) (xy 146.05 85.09)
+			(xy 142.24 91.44) (xy 142.24 85.09)
 		)
 		(stroke
@@
 	(wire
 		(pts
-			(xy 128.27 85.09) (xy 132.08 85.09)
-		)
-		(stroke
-			(width 0)
-			(type default)
-		)
-	)
-	(wire
-		(pts
-			(xy 120.65 97.79) (xy 139.7 97.79)
+			(xy 127 85.09) (xy 128.27 85.09)
+		)
+		(stroke
+			(width 0)
+			(type default)
+		)
+	)
+	(wire
+		(pts
+			(xy 120.65 97.79) (xy 135.89 97.79)
 		)
 		(stroke
@@
 	(wire
 		(pts
-			(xy 128.27 91.44) (xy 146.05 91.44)
-		)
-		(stroke
-			(width 0)
-			(type default)
-		)
-	)
-	(wire
-		(pts
 			(xy 77.47 85.09) (xy 87.63 85.09)
 		)
@@
 	(wire
 		(pts
-			(xy 154.94 90.17) (xy 154.94 97.79)
-		)
-		(stroke
-			(width 0)
-			(type default)
-		)
-	)
-	(wire
-		(pts
-			(xy 111.76 91.44) (xy 128.27 91.44)
-		)
-		(stroke
-			(width 0)
-			(type default)
-		)
-	)
-	(wire
-		(pts
-			(xy 154.94 97.79) (xy 139.7 97.79)
+			(xy 151.13 90.17) (xy 151.13 97.79)
+		)
+		(stroke
+			(width 0)
+			(type default)
+		)
+	)
+	(wire
+		(pts
+			(xy 111.76 91.44) (xy 127 91.44)
+		)
+		(stroke
+			(width 0)
+			(type default)
+		)
+	)
+	(wire
+		(pts
+			(xy 151.13 97.79) (xy 135.89 97.79)
 		)
 		(stroke
@@
 	(wire
 		(pts
-			(xy 128.27 91.44) (xy 128.27 85.09)
-		)
-		(stroke
-			(width 0)
-			(type default)
-		)
-	)
-	(wire
-		(pts
-			(xy 154.94 97.79) (xy 165.1 97.79)
+			(xy 127 91.44) (xy 127 85.09)
+		)
+		(stroke
+			(width 0)
+			(type default)
+		)
+	)
+	(wire
+		(pts
+			(xy 127 91.44) (xy 142.24 91.44)
+		)
+		(stroke
+			(width 0)
+			(type default)
+		)
+	)
+	(wire
+		(pts
+			(xy 151.13 97.79) (xy 161.29 97.79)
 		)
 		(stroke
@@
 	(wire
 		(pts
-			(xy 146.05 85.09) (xy 147.32 85.09)
+			(xy 142.24 85.09) (xy 143.51 85.09)
 		)
 		(stroke
@@
 	(hierarchical_label "BFLOWD"
 		(shape output)
-		(at 165.1 97.79 0)
+		(at 161.29 97.79 0)
 		(effects
 			(font
@@
 		(lib_id "Transistor_FET:Q_NMOS_SSSGD_AvalancheRated")
 		(at 118.11 85.09 0)
+		(mirror x)
 		(unit 1)
 		(exclude_from_sim no)
@@
 		(dnp no)
 		(property "Reference" "Q5"
-			(at 121.92 88.646 0)
+			(at 121.92 88.9 0)
 			(effects
 				(font
@@
 		)
 		(property "Value" "NTMFS5C612NLT1G"
-			(at 111.76 72.39 0)
-			(effects
-				(font
-					(size 1.27 1.27)
-				)
-				(justify left)
+			(at 114.3 74.93 0)
+			(effects
+				(font
+					(size 1.27 1.27)
+				)
 			)
 		)
 		(property "Footprint" "local:DFN-5_L6.1-W5.1-P1.27-BL"
-			(at 123.19 82.55 0)
+			(at 123.19 87.63 0)
 			(effects
 				(font
@@
 	(symbol
 		(lib_id "Transistor_FET:Q_NMOS_SSSGD_AvalancheRated")
-		(at 152.4 85.09 0)
+		(at 133.35 85.09 0)
+		(mirror x)
 		(unit 1)
 		(exclude_from_sim no)
@@
 		(dnp no)
 		(property "Reference" "Q6"
-			(at 155.956 88.9 0)
+			(at 137.16 88.9 0)
 			(effects
 				(font
@@
 		)
 		(property "Value" "NTMFS5C612NLT1G"
-			(at 145.796 72.136 0)
-			(effects
-				(font
-					(size 1.27 1.27)
-				)
-				(justify left)
+			(at 133.35 74.93 0)
+			(effects
+				(font
+					(size 1.27 1.27)
+				)
 			)
 		)
 		(property "Footprint" "local:DFN-5_L6.1-W5.1-P1.27-BL"
-			(at 157.48 82.55 0)
+			(at 138.43 87.63 0)
 			(effects
 				(font
@@
 		)
 		(property "Datasheet" "~"
-			(at 152.4 85.09 0)
+			(at 133.35 85.09 0)
 			(effects
 				(font
@@
 		)
 		(property "Description" "N-MOSFET transistor, source (pins 1-3)/gate/drain (pin 5), SO-8/SO-8F/SO-8FL/SON-8/PowerPAK-8/TDSON-8/VSON-8"
-			(at 152.4 85.09 0)
+			(at 133.35 85.09 0)
 			(effects
 				(font
@@
 		)
 		(property "MPN" "NTMFS5C612NLT1G"
-			(at 152.4 85.09 0)
+			(at 133.35 85.09 0)
 			(effects
 				(font
@@
 		)
 		(property "Desc" "Bflow"
-			(at 152.4 85.09 0)
+			(at 133.35 85.09 0)
 			(effects
 				(font
@@
 		)
 		(property "Manufacturer" ""
-			(at 152.4 85.09 0)
+			(at 133.35 85.09 0)
 			(effects
 				(font
@@
 		)
 		(property "Digikey" ""
-			(at 152.4 85.09 0)
+			(at 133.35 85.09 0)
 			(effects
 				(font
@@
 		)
 		(property "LCSC" "C348543"
-			(at 152.4 85.09 0)
+			(at 133.35 85.09 0)
 			(effects
 				(font
@@
 	(symbol
 		(lib_id "Transistor_FET:Q_NMOS_SSSGD_AvalancheRated")
-		(at 137.16 85.09 0)
+		(at 148.59 85.09 0)
+		(mirror x)
 		(unit 1)
 		(exclude_from_sim no)
@@
 		(dnp no)
 		(property "Reference" "Q7"
-			(at 140.208 88.9 0)
+			(at 152.4 88.9 0)
 			(effects
 				(font
@@
 		)
 		(property "Value" "NTMFS5C612NLT1G"
-			(at 130.302 74.676 0)
-			(effects
-				(font
-					(size 1.27 1.27)
-				)
-				(justify left)
+			(at 152.4 74.93 0)
+			(effects
+				(font
+					(size 1.27 1.27)
+				)
 			)
 		)
 		(property "Footprint" "local:DFN-5_L6.1-W5.1-P1.27-BL"
-			(at 142.24 82.55 0)
+			(at 153.67 87.63 0)
 			(effects
 				(font
@@
 		)
 		(property "Datasheet" "~"
-			(at 137.16 85.09 0)
+			(at 148.59 85.09 0)
 			(effects
 				(font
@@
 		)
 		(property "Description" "N-MOSFET transistor, source (pins 1-3)/gate/drain (pin 5), SO-8/SO-8F/SO-8FL/SON-8/PowerPAK-8/TDSON-8/VSON-8"
-			(at 137.16 85.09 0)
+			(at 148.59 85.09 0)
 			(effects
 				(font
@@
 		)
 		(property "MPN" "NTMFS5C612NLT1G"
-			(at 137.16 85.09 0)
+			(at 148.59 85.09 0)
 			(effects
 				(font
@@
 		)
 		(property "Desc" "Bflow"
-			(at 137.16 85.09 0)
+			(at 148.59 85.09 0)
 			(effects
 				(font
@@
 		)
 		(property "Manufacturer" ""
-			(at 137.16 85.09 0)
+			(at 148.59 85.09 0)
 			(effects
 				(font
@@
 		)
 		(property "Digikey" ""
-			(at 137.16 85.09 0)
+			(at 148.59 85.09 0)
 			(effects
 				(font
@@
 		)
 		(property "LCSC" "C348543"
-			(at 137.16 85.09 0)
-			(effects
-				(font
+			(at 148.59 85.09 0)
+			(effects
+				(font
